Commit message: Updating the UTM and ECEF coordinates on all files.

File: stacks/squirtle_robot/trunk/squirtle_description/urdf/mondego_river.urdf (robot description, URDF)
Before this commit: robot mondego_river, 3 links, 2 joints
Links:
- removed link base_station
- added link mondego; visual box size=346.0 346.0 10.0
- link world: geometry visual box size=0.001 0.001 0.001
Joints:
- removed joint world_base_station_joint
- removed joint world_bridge_joint
- added joint mondego_bridge_joint: type fixed, parent mondego, child bridge, origin xyz=70 15 5 rpy=0 0 1.66
- added joint world_mondego_joint: type fixed, parent world, child mondego, origin xyz=548811.454358155 4450122.57607714 0 rpy=0 0 0

Commit message: Minor bugs after testing in the river.

File: stacks/squirtle_robot/trunk/squirtle_description/urdf/mondego_river.urdf (robot description, URDF)
Before this commit: robot mondego_river, 3 links, 2 joints
Joints:
- joint world_mondego_joint: origin xyz=548811.454358155 4450122.57607714 0 rpy=0 0 0 -> xyz=548811.454358155 4450122.57607714 0 rpy=0 0 1.57

File: stacks/squirtle_robot/trunk/squirtle_description/urdf/squirtle.urdf (robot description, URDF)
Before this commit: robot squirtle, 7 links, 6 joints
Links:
- added link gps; visual mesh filename=package://squirtle_description/meshes/gps_antenna.dae
Joints:
- added joint gps_joint: type fixed, parent base_link, child gps, origin xyz=-0.24 -0.2 0.25 rpy=0 0 0
- joint base_footprint_base_link_joint: axis 0 0 1 -> (none)
- joint cyclops_joint: axis 0 0 1 -> (none)
- joint imu_joint: axis 0 0 1 -> (none)
- joint sonar_joint: axis 0 0 1 -> (none)
