Commit message: Updating the isr and mondego urdf files for a 0 height.

File: stacks/squirtle_robot/trunk/squirtle_description/urdf/isr.urdf (robot description, URDF)
Before this commit: robot isr_garage, 2 links, 1 joints
Links:
- link isr: geometry visual box size=60.0 50.0 0.0

File: stacks/squirtle_robot/trunk/squirtle_description/urdf/mondego_river.urdf (robot description, URDF)
Before this commit: robot mondego_river, 3 links, 2 joints
Links:
- link mondego: geometry visual box size=346.0 346.0 0.0
